Commit message: visual simplified shape

File: hardware/URDF/robots/Poppy_Humanoid.URDF (robot description, URDF)
Before this commit: robot Poppy_Humanoid, 26 links, 25 joints
Links:
- link abdomen: geometry collision mesh filename=package://meshes/abdomen_respondable.STL; visual mesh filename=package://meshes/abdomen_visual.STL
- link abs_motors: geometry collision mesh filename=package://meshes/abs_motors_respondable.STL; visual mesh filename=package://meshes/abs_motors_visual.STL
- link bust_motors: geometry collision mesh filename=package://meshes/bust_motors_respondable.STL; visual mesh filename=package://meshes/bust_motors_visual.STL
- link chest: geometry collision mesh filename=package://meshes/chest_respondable.STL; visual mesh filename=package://meshes/chest_visual.STL
- link head: geometry collision mesh filename=package://meshes/head_respondable.STL; visual mesh filename=package://meshes/head_visual.STL
- link l_foot: geometry collision mesh filename=package://meshes/l_foot_respondable.STL; visual mesh filename=package://meshes/l_foot_visual.STL
- link l_forearm: geometry collision mesh filename=package://meshes/l_forearm_respondable.STL; visual mesh filename=package://meshes/l_forearm_visual.STL
- link l_hip: geometry collision mesh filename=package://meshes/l_hip_respondable.STL; visual mesh filename=package://meshes/l_hip_visual.STL
- link l_hip_motor: geometry collision mesh filename=package://meshes/l_hip_motor_respondable.STL; visual mesh filename=package://meshes/l_hip_motor_visual.STL
- link l_shin: geometry collision mesh filename=package://meshes/l_shin_respondable.STL; visual mesh filename=package://meshes/l_shin_visual.STL
- link l_shoulder: geometry collision mesh filename=package://meshes/l_shoulder_respondable.STL; visual mesh filename=package://meshes/l_shoulder_visual.STL
- link l_shoulder_motor: geometry collision mesh filename=package://meshes/l_shoulder_motor_respondable.STL; visual mesh filename=package://meshes/l_shoulder_motor_visual.STL
- link l_thigh: geometry collision mesh filename=package://meshes/l_thigh_respondable.STL; visual mesh filename=package://meshes/l_thigh_visual.STL
- link l_upper_arm: geometry collision mesh filename=package://meshes/l_upper_arm_respondable.STL; visual mesh filename=package://meshes/l_upper_arm_visual.STL
- link neck: geometry collision mesh filename=package://meshes/neck_respondable.STL; visual mesh filename=package://meshes/neck_visual.STL
- link pelvis: geometry collision mesh filename=package://meshes/pelvis_respondable.STL; visual mesh filename=package://meshes/pelvis_visual.STL
- link r_foot: geometry collision mesh filename=package://meshes/r_foot_respondable.STL; visual mesh filename=package://meshes/r_foot_visual.STL
- link r_forearm: geometry collision mesh filename=package://meshes/r_forearm_respondable.STL; visual mesh filename=package://meshes/r_forearm_visual.STL
- link r_hip: geometry collision mesh filename=package://meshes/r_hip_respondable.STL; visual mesh filename=package://meshes/r_hip_visual.STL
- link r_hip_motor: geometry collision mesh filename=package://meshes/r_hip_motor_respondable.STL; visual mesh filename=package://meshes/r_hip_motor_visual.STL
- link r_shin: geometry collision mesh filename=package://meshes/r_shin_respondable.STL; visual mesh filename=package://meshes/r_shin_visual.STL
- link r_shoulder: geometry collision mesh filename=package://meshes/r_shoulder_respondable.STL; visual mesh filename=package://meshes/r_shoulder_visual.STL
- link r_shoulder_motor: geometry collision mesh filename=package://meshes/r_shoulder_motor_respondable.STL; visual mesh filename=package://meshes/r_shoulder_motor_visual.STL
- link r_thigh: geometry collision mesh filename=package://meshes/r_thigh_respondable.STL; visual mesh filename=package://meshes/r_thigh_visual.STL
- link r_upper_arm: geometry collision mesh filename=package://meshes/r_upper_arm_respondable.STL; visual mesh filename=package://meshes/r_upper_arm_visual.STL
- link spine: geometry collision mesh filename=package://meshes/spine_respondable.STL; visual mesh filename=package://meshes/spine_visual.STL
