Commit message: base meshs added, urdf modified for stl ext

File: hardware/URDF/robots/Poppy_Torso.URDF (robot description, URDF)
Before this commit: robot Poppy_Torso, 14 links, 13 joints
Links:
- link bust_motors: geometry collision mesh filename=package://Poppy_Torso/meshes/bust_motors_respondable.stl; visual mesh filename=package://Poppy_Torso/meshes/bust_motors_visual.STL
- link head: geometry collision mesh filename=package://Poppy_Torso/meshes/head_respondable.stl; visual mesh filename=package://Poppy_Torso/meshes/head_visual.STL
- link l_forearm: geometry collision mesh filename=package://Poppy_Torso/meshes/l_forearm_respondable.stl; visual mesh filename=package://Poppy_Torso/meshes/l_forearm_visual.STL
- link l_shoulder: geometry collision mesh filename=package://Poppy_Torso/meshes/l_shoulder_respondable.stl; visual mesh filename=package://Poppy_Torso/meshes/l_shoulder_visual.STL
- link l_shoulder_motor: geometry collision mesh filename=package://Poppy_Torso/meshes/l_shoulder_motor_respondable.s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; visual mesh filename=package://Poppy_Torso/meshes/l_shoulder_motor_visual.STL

Commit message: optimized V-REP scene for inertia and PID

File: hardware/URDF/robots/Poppy_Torso.URDF (robot description, URDF)
Before this commit: robot Poppy_Torso, 14 links, 13 joints
Links:
- link base: geometry collision mesh filename=package://meshes/base_respondable.STL; visual mesh filename=package://meshes/base_visual.STL
- link bust_motors: mass 0.158876054417129 -> 0.158876054570625; geometry collision mesh filename=package://meshes/bust_motors_respondable.STL; visual mesh filename=package://meshes/bust_motors_visual.STL
- link chest: mass 0.262924546647766 -> 0.262925523172723; geometry collision mesh filename=package://meshes/chest_respondable.STL; visual mesh filename=package://meshes/chest_visual.STL
- link head: mass 0.188564677402165 -> 0.188564323997503; geometry collision mesh filename=package://meshes/head_respondable.STL; visual mesh filename=package://meshes/head_visual.STL
- link l_forearm: mass 0.0486517775557926 -> 0.0486512481725727; geometry collision mesh filename=package://meshes/l_forearm_respondable.STL; visual mesh filename=package://meshes/l_forearm_visual.STL
- link l_shoulder: mass 0.00843598833388653 -> 0.00843598968780806; geometry collision mesh filename=package://meshes/l_shoulder_respondable.STL; visual mesh filename=package://meshes/l_shoulder_visual.STL
- link l_shoulder_motor: mass 0.082814411658021 -> 0.0828144098443214; geometry collision mesh filename=package://meshes/l_shoulder_motor_respondable.STL; visual mesh filename=package://meshes/l_shoulder_motor_visual.STL
- link neck: mass 0.00588496516988366 -> 0.00588496516988365; geometry collision mesh filename=package://meshes/neck_respondable.STL; visual mesh filename=package://meshes/neck_visual.STL
- link r_forearm: mass 0.0486519712384455 -> 0.0486511084909604; geometry collision mesh filename=package://meshes/r_forearm_respondable.STL; visual mesh filename=package://meshes/r_forearm_visual.STL
- link r_shoulder: mass 0.00848189595252892 -> 0.00848189714003649; geometry collision mesh filename=package://meshes/r_shoulder_respondable.STL; visual mesh filename=package://meshes/r_shoulder_visual.STL
- link r_shoulder_motor: mass 0.0828144642064673 -> 0.0828144098443213; geometry collision mesh filename=package://meshes/r_shoulder_motor_respondable.STL; visual mesh filename=package://meshes/r_shoulder_motor_visual.STL
- link spine: mass 0.0926815111299683 -> 0.0926815106655512; geometry collision mesh filename=package://meshes/spine_respondable.STL; visual mesh filename=package://meshes/spine_visual.STL
Joints:
- joint bust_y: limit lower=-0.802851455917 upper=0.401425727959 effort=3.1 velocity=7.0 -> lower=-1.16937059884 upper=0.471238898038 effort=3.1 velocity=7.0
- joint head_y: limit lower=-0.698131700798 upper=0.13962634016 effort=1.8 velocity=10.0 -> lower=-0.785398163397 upper=0.10471975512 effort=1.8 velocity=10.0
- joint head_z: limit lower=-1.74532925199 upper=1.74532925199 effort=1.8 velocity=10.0 -> lower=-1.57079632679 upper=1.57079632679 effort=1.8 velocity=10.0
- joint l_arm_z: limit lower=-1.57079632679 upper=1.57079632679 effort=3.1 velocity=7.0 -> lower=-1.83259571459 upper=1.83259571459 effort=3.1 velocity=7.0
- joint l_elbow_y: limit lower=-2.44346095279 upper=0.0 effort=3.1 velocity=7.0 -> lower=-2.58308729295 upper=0.0174532925199 effort=3.1 velocity=7.0
- joint r_arm_z: limit lower=-1.57079632679 upper=1.57079632679 effort=3.1 velocity=7.0 -> lower=-1.83259571459 upper=1.83259571459 effort=3.1 velocity=7.0
- joint r_elbow_y: limit lower=0.0 upper=2.56563400043 effort=3.1 velocity=7.0 -> lower=-0.0174532925199 upper=2.58308729295 effort=3.1 velocity=7.0
